File: untitled.kicad_sch (KiCad schematic)
At the start: 138 parts, among them SW10 SW_Push, SW11 SW_Push, SW12 SW_Push, SW13 SW_Push, SW14 SW_Push, SW15 SW_Push, SW16 SW_Push, SW17 SW_Push, SW18 SW_Push, SW19 SW_Push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

Commit message: fix names
Other:
- title: (none) -> Switch Matrix
Changed lines of the file:
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@@
 	(generator_version "9.0")
 	(paper "User" 635 279.4)
+	(title_block
+		(title "Switch Matrix")
+	)
 	(junction
 		(at 238.76 130.81)
