File: Keyboard.kicad_sch (KiCad schematic)
At the start: 18 parts, among them J1 USB_C_Receptacle_USB2.0_16P, J2 Conn_01x04, SW1 SW_Push, U1 ATmega32U4-A, U2 USB6B1, Y1 Crystal_GND24_Small

Commit message: name fix
Other:
- sheet Switch Matrix: file untitled.kicad_sch -> Switch_Matrix.kicad_sch
- title: Keyboard -> Switch Matrix
Changed lines of the file:
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@@
 	(paper "A4")
 	(title_block
-		(title "Keyboard")
+		(title "Switch Matrix")
 		(company "Darren Lin")
 		(comment 1 "65% keyboard")
@@
 	)
 	(sheet
-		(at 151.765 186.055)
+		(at 146.685 187.325)
 		(size 12.7 3.81)
 		(exclude_from_sim no)
@@
 		)
 		(property "Sheetname" "Switch Matrix"
-			(at 151.765 185.3434 0)
+			(at 146.685 186.6134 0)
 			(effects
 				(font
@@
 			)
 		)
-		(property "Sheetfile" "untitled.kicad_sch"
-			(at 151.765 190.4496 0)
+		(property "Sheetfile" "Switch_Matrix.kicad_sch"
+			(at 146.685 191.7196 0)
 			(effects
 				(font
