File: Kicad/_autosave-Keyboard.kicad_pcb (KiCad board)
At the start: 2 copper layers, 324 x 97 mm, 171 parts, among them J1 USB_C_Receptacle_USB2.0_16P, J2 Conn_01x04, SW10 SW_Push, SW11 SW_Push, SW12 SW_Push, SW13 SW_Push, SW14 SW_Push, SW15 SW_Push, SW16 SW_Push, SW17 SW_Push, SW18 SW_Push, SW19 SW_Push, SW2 SW_Push, SW20 SW_Push, SW21 SW_Push, SW22 SW_Push, SW23 SW_Push, SW24 SW_Push, SW25 SW_Push, SW26 SW_Push, SW27 SW_Push, SW28 SW_Push, SW29 SW_Push, SW3 SW_Push, SW30 SW_Push, SW31 SW_Push, SW32 SW_Push, SW33 SW_Push, SW34 SW_Push, SW35 SW_Push, SW36 SW_Push, SW37 SW_Push, SW38 SW_Push, SW39 SW_Push, SW4 SW_Push, SW40 SW_Push, SW41 SW_Push, SW42 SW_Push, SW43 SW_Push, SW44 SW_Push, SW45 SW_Push, SW46 SW_Push, SW47 SW_Push, SW48 SW_Push, SW49 SW_Push, SW5 SW_Push, SW50 SW_Push, SW51 SW_Push, SW52 SW_Push, SW53 SW_Push, SW54 SW_Push, SW55 SW_Push, SW56 SW_Push, SW57 SW_Push, SW58 SW_Push, SW59 SW_Push, SW6 SW_Push, SW60 SW_Push, SW61 SW_Push, SW62 SW_Push, SW63 SW_Push, SW64 SW_Push, SW65 SW_Push, SW66 SW_Push, SW67 SW_Push, SW68 SW_Push, SW69 SW_Push, SW7 SW_Push, SW70 SW_Push, SW71 RotaryEncoder_Switch, SW8 SW_Push, SW9 SW_Push, U1 ATmega32U4-A, U2 USB6B1, Y1 Crystal_GND24_Small

Commit message: fixed edge cuts/mounting holes + board review
Parts:
- moved J1 2.00 mm to (49.6, 29.8)
Routing:
- net GND: track 22.3 -> 26.8 mm
- net VBUS: track 437.1 -> 439.3 mm
- net Net-(J1-CC1): track 2.88 -> 5.00 mm
- net Net-(J1-CC2): track 5.56 -> 7.68 mm
- net Net-(J1-D--PadA7): track 12.4 -> 14.4 mm
- net Net-(J1-D+-PadA6): track 12.4 -> 14.0 mm
Other:
- board size 324 x 97 mm -> 327 x 99 mm
