File: Kicad/_autosave-Keyboard.kicad_pcb (KiCad board)
At the start: 2 copper layers, 327 x 99 mm, 177 parts, among them J1 USB_C_Receptacle_USB2.0_16P, J2 Conn_01x04, SW10 SW_Push, SW11 SW_Push, SW12 SW_Push, SW13 SW_Push, SW14 SW_Push, SW15 SW_Push, SW16 SW_Push, SW17 SW_Push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

Commit message: stitching vias
Routing:
- net GND: vias 2 -> 251
Other:
- outline, holes or cut-outs redrawn
