File: Kicad/Keyboard.kicad_pcb (KiCad board)
At the start: 2 copper layers, 324 x 97 mm, 171 parts, among them J1 USB_C_Receptacle_USB2.0_16P, J2 Conn_01x04, SW10 SW_Push, SW11 SW_Push, SW12 SW_Push, SW13 SW_Push, SW14 SW_Push, SW15 SW_Push, SW16 SW_Push, SW17 SW_Push, SW18 SW_Push, SW19 SW_Push, SW2 SW_Push, SW20 SW_Push, SW21 SW_Push, SW22 SW_Push, SW23 SW_Push, SW24 SW_Push, SW25 SW_Push, SW26 SW_Push, SW27 SW_Push, SW28 SW_Push, SW29 SW_Push, SW3 SW_Push, SW30 SW_Push, SW31 SW_Push, SW32 SW_Push, SW33 SW_Push, SW34 SW_Push, SW35 SW_Push, SW36 SW_Push, SW37 SW_Push, SW38 SW_Push, SW39 SW_Push, SW4 SW_Push, SW40 SW_Push, SW41 SW_Push, SW42 SW_Push, SW43 SW_Push, SW44 SW_Push, SW45 SW_Push, SW46 SW_Push, SW47 SW_Push, SW48 SW_Push, SW49 SW_Push, SW5 SW_Push, SW50 SW_Push, SW51 SW_Push, SW52 SW_Push, SW53 SW_Push, SW54 SW_Push, SW55 SW_Push, SW56 SW_Push, SW57 SW_Push, SW58 SW_Push, SW59 SW_Push, SW6 SW_Push, SW60 SW_Push, SW61 SW_Push, SW62 SW_Push, SW63 SW_Push, SW64 SW_Push, SW65 SW_Push, SW66 SW_Push, SW67 SW_Push, SW68 SW_Push, SW69 SW_Push, SW7 SW_Push, SW70 SW_Push, SW71 RotaryEncoder_Switch, SW8 SW_Push, SW9 SW_Push, U1 ATmega32U4-A, U2 USB6B1, Y1 Crystal_GND24_Small

Commit message: differential routing + board review
Parts:
- moved J1 2.00 mm to (49.6, 29.8)
- moved R1 1.86 mm to (49.4, 53.0)
- moved R2 1.55 mm to (50.7, 53.0)
- moved C2 0.93 mm to (45.3, 61.6)
Connections:
- J1 pad A6: Net-(J1-D+-PadA6) -> D1_+
- J1 pad A7: Net-(J1-D--PadA7) -> D1_-
- J1 pad B6: Net-(J1-D+-PadA6) -> D1_+
- J1 pad B7: Net-(J1-D--PadA7) -> D1_-
- J1 pad S1: unconnected-(J1-SHIELD-PadS1)_1 -> GND
- R1 pad 1: D+ -> Net-(R1-Pad1)
- R1 pad 2: Net-(U1-D+) -> D+
- R2 pad 1: Net-(U1-D-) -> D-
- R2 pad 2: D- -> Net-(R2-Pad2)
- U1 pad 3: Net-(U1-D-) -> D-
- U1 pad 4: Net-(U1-D+) -> D+
- U2 pad 2: Net-(J1-D--PadA7) -> D1_+
- U2 pad 3: Net-(J1-D+-PadA6) -> D1_-
- U2 pad 6: D+ -> Net-(R2-Pad2)
- U2 pad 7: D- -> Net-(R1-Pad1)
- Y1 pad 1: GND -> Net-(U1-XTAL2)
- Y1 pad 2: Net-(U1-XTAL2) -> GND
- Y1 pad 3: GND -> Net-(U1-XTAL1)
- Y1 pad 4: Net-(U1-XTAL1) -> GND
Routing:
- net D1_-: track 0.00 -> 25.6 mm
- net D1_+: track 0.00 -> 23.1 mm
- net Net-(U1-D-): track 19.1 -> 0.00 mm, vias 2 -> 0
- net Net-(U1-D+): track 17.1 -> 0.00 mm, vias 2 -> 0
- net D-: track 2.29 -> 18.9 mm, vias 0 -> 2
- net D+: track 2.35 -> 18.9 mm, vias 0 -> 2
- net Net-(J1-D--PadA7): track 12.4 -> 0.00 mm
- net Net-(J1-D+-PadA6): track 12.4 -> 0.00 mm
- net GND: track 22.3 -> 31.5 mm, vias 0 -> 2
- net Net-(U1-XTAL2): track 19.0 -> 15.3 mm
- net C7: track 236.7 -> 239.4 mm
- net Net-(U1-XTAL1): track 11.3 -> 13.7 mm, vias 2 -> 0
- net Net-(R2-Pad2): track 0.00 -> 2.32 mm
- net Net-(R1-Pad1): track 0.00 -> 2.31 mm
- net Net-(J1-CC1): track 2.88 -> 5.00 mm
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Other:
- board size 324 x 97 mm -> 327 x 99 mm

Commit message: fix mounting holes finalizing stuff
Parts:
- added M.2: MountingHole_2.2mm_M2_ISO14580, MountingHole:MountingHole_2.2mm_M2_ISO14580, F.Cu at (266.3, 98.5)
- added M.2: MountingHole_2.2mm_M2_ISO14580, MountingHole:MountingHole_2.2mm_M2_ISO14580, F.Cu at (69.6, 97.0)
- added M.2: MountingHole_2.2mm_M2_ISO14580, MountingHole:MountingHole_2.2mm_M2_ISO14580, F.Cu at (288.8, 55.9)
- added M.2: MountingHole_2.2mm_M2_ISO14580, MountingHole:MountingHole_2.2mm_M2_ISO14580, F.Cu at (121.2, 118.8)
- added M.2: MountingHole_2.2mm_M2_ISO14580, MountingHole:MountingHole_2.2mm_M2_ISO14580, F.Cu at (133.5, 65.7)
- added M.2: MountingHole_2.2mm_M2_ISO14580, MountingHole:MountingHole_2.2mm_M2_ISO14580, F.Cu at (198.8, 118.8)
Other:
- outline, holes or cut-outs redrawn
