File: Kicad/Keyboard.kicad_pcb (KiCad board)
At the start: 2 copper layers, 327 x 99 mm, 177 parts, among them J1 USB_C_Receptacle_USB2.0_16P, J2 Conn_01x04, SW10 SW_Push, SW11 SW_Push, SW12 SW_Push, SW13 SW_Push, SW14 SW_Push, SW15 SW_Push, SW16 SW_Push, SW17 SW_Push, SW18 SW_Push, SW19 SW_Push, SW2 SW_Push, SW20 SW_Push, SW21 SW_Push, SW22 SW_Push, SW23 SW_Push, SW24 SW_Push, SW25 SW_Push, SW26 SW_Push, SW27 SW_Push, SW28 SW_Push, SW29 SW_Push, SW3 SW_Push, SW30 SW_Push, SW31 SW_Push, SW32 SW_Push, SW33 SW_Push, SW34 SW_Push, SW35 SW_Push, SW36 SW_Push, SW37 SW_Push, SW38 SW_Push, SW39 SW_Push, SW4 SW_Push, SW40 SW_Push, SW41 SW_Push, SW42 SW_Push, SW43 SW_Push, SW44 SW_Push, SW45 SW_Push, SW46 SW_Push, SW47 SW_Push, SW48 SW_Push, SW49 SW_Push, SW5 SW_Push, SW50 SW_Push, SW51 SW_Push, SW52 SW_Push, SW53 SW_Push, SW54 SW_Push, SW55 SW_Push, SW56 SW_Push, SW57 SW_Push, SW58 SW_Push, SW59 SW_Push, SW6 SW_Push, SW60 SW_Push, SW61 SW_Push, SW62 SW_Push, SW63 SW_Push, SW64 SW_Push, SW65 SW_Push, SW66 SW_Push, SW67 SW_Push, SW68 SW_Push, SW69 SW_Push, SW7 SW_Push, SW70 SW_Push, SW71 RotaryEncoder_Switch, SW8 SW_Push, SW9 SW_Push, U1 ATmega32U4-A, U2 USB6B1, Y1 Crystal_GND24_Small

Commit message: caught huge mcu i2c issue
Connections:
- U1 pad 1: R3 -> R1
- U1 pad 18: C10 -> SCL
- U1 pad 19: C11 -> SDA
- U1 pad 20: C12 -> C10
- U1 pad 21: C13 -> C11
- U1 pad 22: R0 -> C13
- U1 pad 25: C14 -> C12
- U1 pad 26: R1 -> C14
- U1 pad 27: R2 -> R0
- U1 pad 39: SDA -> R4
- U1 pad 40: SCL -> R3
- U1 pad 41: R4 -> R2
Routing:
- net SDA: track 305.4 -> 321.3 mm, vias 0 -> 2
- net R1: track 294.5 -> 309.7 mm, vias 0 -> 4
- net SCL: track 310.7 -> 319.6 mm, vias 0 -> 4
- net R2: track 305.7 -> 297.7 mm
- net C11: track 325.5 -> 318.4 mm, vias 5 -> 3
- net C12: track 331.2 -> 324.4 mm
- net R3: track 328.5 -> 334.0 mm, vias 2 -> 4
- net C10: track 300.2 -> 295.1 mm
- net R4: track 351.7 -> 356.0 mm, vias 2 -> 4
- net R0: track 322.6 -> 326.4 mm, vias 4 -> 2
- net C13: track 348.3 -> 351.3 mm
- net GND: track 31.5 -> 33.2 mm
- net C14: track 360.9 -> 361.1 mm, vias 27 -> 3
